Commit message: Add and modify files

File: src/amrbot_description/urdf/modules/base.xacro (robot description, xacro)
@@ -328,5 +328,5 @@
     <parent link="motor_assy_2_link"/>
     <child link="wheel_assy_2_link"/>
-    <axis xyz="0 0 1"/>
+    <axis xyz="0 0 -1"/>
     <limit effort="10" velocity="10"/>
   </joint>

File: src/amrbot_description/urdf/modules/imu.xacro (robot description, xacro)
@@ -27,5 +27,5 @@
   <!-- Joint from base_link to imu -->
   <joint name="imu_joint" type="fixed">
-    <origin xyz="0.00275956 0.00314761 0.0133316" rpy="3.14159 -0 0"/>
+    <origin xyz="0.00275956 0.00314761 0.0133316" rpy="0 0 3.14159"/>
     <parent link="base_link"/>
     <child link="imu_link"/>

File: src/amrbot_description/urdf/xacro_properties/xacro_properties.xacro (robot description, xacro)
@@ -2,4 +2,4 @@
 <robot xmlns:xacro="http://www.ros.org/wiki/xacro">
     <xacro:property name="package_name" value="amrbot_description"/>
-    <xacro:property name="robot_name" value="amr_bot"/>
+    <xacro:property name="robot_name" value="amrbot"/>
 </robot>

File: src/amrbot_gazebo/urdf/gazebo_plugins.xacro (robot description, xacro)
@@ -1,7 +1,4 @@
 <?xml version="1.0" ?>
-<!-- Generated using onshape-to-robot -->
-<!-- Onshape https://cad.onshape.com/documents/4209ac7f0152411e9d4dcbf0/w/3377871fe4109e8e8f25bc5b/e/d6705610344c69e12c64875a -->
 <robot xmlns:xacro="http://www.ros.org/wiki/xacro">
-    <!-- ==================== GLOBAL SENSOR PLUGINS (MANDATORY FOR IMU) ==================== -->
     <gazebo>
         <plugin filename="gz-sim-sensors-system" name="gz::sim::systems::Sensors">
@@ -11,32 +8,29 @@
         </plugin>
     </gazebo>
-    <!-- ==================== DIFF DRIVE PLUGIN ==================== -->
     <gazebo>
         <plugin filename="gz-sim-diff-drive-system" name="gz::sim::systems::DiffDrive">
             <left_joint>left_wheel_joint</left_joint>
             <right_joint>right_wheel_joint</right_joint>
-            <wheel_separation>0.3306</wheel_separation>
-            <wheel_radius>0.05675</wheel_radius>
+            <wheel_separation>0.4776</wheel_separation>
+            <wheel_radius>0.05895</wheel_radius>
             <topic>/cmd_vel</topic>
             <odom_topic>/odom</odom_topic>
-            <tf_topic>/tf</tf_topic>
             <frame_id>odom</frame_id>
             <child_frame_id>base_footprint</child_frame_id>
-            <odometry_frame>odom</odometry_frame>
             <max_linear_velocity>1.0</max_linear_velocity>
             <max_linear_acceleration>0.5</max_linear_acceleration>
         </plugin>
     </gazebo>
-    <!-- ==================== JOINT STATE PUBLISHER ==================== -->
     <gazebo>
         <plugin filename="gz-sim-joint-state-publisher-system" name="gz::sim::systems::JointStatePublisher">
-            <joint_name>wheel_left_joint</joint_name>
-            <joint_name>wheel_right_joint</joint_name>
-            <joint_name>caster_wheel_left_joint</joint_name>
-            <joint_name>caster_wheel_right_joint</joint_name>
+            <joint_name>left_wheel_joint</joint_name>
+            <joint_name>right_wheel_joint</joint_name>
+            <joint_name>lf_caster_wheel_joint</joint_name>
+            <joint_name>lb_caster_wheel_joint</joint_name>
+            <joint_name>rf_caster_wheel_joint</joint_name>
+            <joint_name>rb_caster_wheel_joint</joint_name>
             <topic>joint_states</topic>
         </plugin>
     </gazebo>
-    <!-- ==================== IMU SENSOR INSTANCE ==================== -->
     <gazebo reference="imu_link">
         <sensor name="imu_sensor" type="imu">

File: src/amrbot_gazebo/urdf/gazebo_properties.xacro (robot description, xacro)
@@ -1,10 +1,7 @@
 <?xml version="1.0" ?>
-<!-- Generated using onshape-to-robot -->
-<!-- Onshape https://cad.onshape.com/documents/4209ac7f0152411e9d4dcbf0/w/3377871fe4109e8e8f25bc5b/e/d6705610344c69e12c64875a -->
 <robot xmlns:xacro="http://www.ros.org/wiki/xacro">
-    <!-- Gazebo properties for the base link -->
     <gazebo reference="base_link">
-        <mu1 value="0.5"/> <!-- Friction coefficient in the first direction -->
-        <mu2 value="0.5"/> <!-- Friction coefficient in the second direction -->
+        <mu1 value="0.5"/>
+        <mu2 value="0.5"/>
     </gazebo>
     <gazebo reference="lidar_link">
@@ -16,15 +13,12 @@
         <mu2 value="0.5"/>
     </gazebo>
-    <!-- ===== LEFT DRIVE WHEEL (higher friction) ===== -->
     <gazebo reference="wheel_assy_link">
         <mu1 value="1.5"/>
         <mu2 value="1.5"/>
     </gazebo>
-    <!-- ===== RIGHT DRIVE WHEEL (higher friction) ===== -->
     <gazebo reference="wheel_assy_2_link">
         <mu1 value="1.5"/>
         <mu2 value="1.5"/>
     </gazebo>
-    <!-- ===== CASTER WHEELS (moderate friction) ===== -->
     <gazebo reference="caster_wheel_link">
         <mu1 value="0.8"/>
