Commit message: modify and delete

File: src/amrbot_description/urdf/amrbot_description.urdf.xacro (robot description, xacro)
@@ -1,6 +1,8 @@
 <?xml version="1.0" ?>
-<robot name="mini_agv" xmlns:xacro="http://www.ros.org/wiki/xacro">
+<robot name="amrbot" xmlns:xacro="http://www.ros.org/wiki/xacro">
   <xacro:arg name="sim" default="false"/>
-  <xacro:include filename="xacro_properties/xacro_properties.xacro"/>
+  <xacro:property name="package_name" value="amrbot_description"/>
+  <xacro:property name="robot_name" value="amrbot"/>
+  <xacro:property name="base_height" value="0.1" />
   <xacro:include filename="modules/base.xacro"/>
   <xacro:include filename="modules/imu.xacro"/>

File: src/amrbot_description/urdf/modules/base.xacro (robot description, xacro)
@@ -8,5 +8,5 @@
         <parent link="base_footprint"/>
         <child link="base_link"/>
-        <origin xyz="0.0 0.0 0.0" rpy="0.0 0.0 0.0"/>
+        <origin xyz="0.0 0.0 ${base_height}" rpy="0.0 0.0 0.0"/>
     </joint>
 <!-- From ONSHAPE -->
@@ -22,5 +22,5 @@
       <origin xyz="0.00275956 0.00314761 -0.00866843" rpy="0 -0 0"/>
       <geometry>
-        <mesh filename="package://amrbot_description/meshes/base_frame.stl"/>
+        <mesh filename="package://${package_name}/meshes/base_frame.stl"/>
       </geometry>
       <material name="base_frame_material">
@@ -31,5 +31,5 @@
       <origin xyz="0.00275956 0.00314761 -0.00866843" rpy="0 -0 0"/>
       <geometry>
-        <mesh filename="package://amrbot_description/meshes/base_frame.stl"/>
+        <mesh filename="package://${package_name}/meshes/base_frame.stl"/>
       </geometry>
     </collision>
@@ -38,5 +38,5 @@
       <origin xyz="0.00275956 0.00314761 -0.00866843" rpy="0 -0 0"/>
       <geometry>
-        <mesh filename="package://amrbot_description/meshes/pvc.stl"/>
+        <mesh filename="package://${package_name}/meshes/pvc.stl"/>
       </geometry>
       <material name="pvc_material">
@@ -47,5 +47,5 @@
       <origin xyz="0.00275956 0.00314761 -0.00866843" rpy="0 -0 0"/>
       <geometry>
-        <mesh filename="package://amrbot_description/meshes/pvc.stl"/>
+        <mesh filename="package://${package_name}/meshes/pvc.stl"/>
       </geometry>
     </collision>
@@ -62,5 +62,5 @@
       <origin xyz="0 -0.007 -0.023" rpy="1.5708 -1.5708 0"/>
       <geometry>
-        <mesh filename="package://amrbot_description/meshes/pg36_body.stl"/>
+        <mesh filename="package://${package_name}/meshes/pg36_body.stl"/>
       </geometry>
       <material name="pg36_body_material">
@@ -71,5 +71,5 @@
       <origin xyz="0 -0.007 -0.023" rpy="1.5708 -1.5708 0"/>
       <geometry>
-        <mesh filename="package://amrbot_description/meshes/pg36_body.stl"/>
+        <mesh filename="package://${package_name}/meshes/pg36_body.stl"/>
       </geometry>
     </collision>
@@ -78,5 +78,5 @@
       <origin xyz="0 -0.0072 -0.023" rpy="-1.5708 -0 0"/>
       <geometry>
-        <mesh filename="package://amrbot_description/meshes/bracket_body.stl"/>
+        <mesh filename="package://${package_name}/meshes/bracket_body.stl"/>
       </geometry>
       <material name="bracket_body_material">
@@ -87,5 +87,5 @@
       <origin xyz="0 -0.0072 -0.023" rpy="-1.5708 -0 0"/>
       <geometry>
-        <mesh filename="package://amrbot_description/meshes/bracket_body.stl"/>
+        <mesh filename="package://${package_name}/meshes/bracket_body.stl"/>
       </geometry>
     </collision>
@@ -94,5 +94,5 @@
       <origin xyz="0 -0.01 -0.023" rpy="-1.5708 -0 0"/>
       <geometry>
-        <mesh filename="package://amrbot_description/meshes/bracket_shaft.stl"/>
+        <mesh filename="package://${package_name}/meshes/bracket_shaft.stl"/>
       </geometry>
       <material name="bracket_shaft_material">
@@ -103,5 +103,5 @@
       <origin xyz="0 -0.01 -0.023" rpy="-1.5708 -0 0"/>
       <geometry>
-        <mesh filename="package://amrbot_description/meshes/bracket_shaft.stl"/>
+        <mesh filename="package://${package_name}/meshes/bracket_shaft.stl"/>
       </geometry>
     </collision>
@@ -110,5 +110,5 @@
       <origin xyz="0 -0.007 -0.023" rpy="1.5708 -1.5708 0"/>
       <geometry>
-        <mesh filename="package://amrbot_description/meshes/pg36_shaft.stl"/>
+        <mesh filename="package://${package_name}/meshes/pg36_shaft.stl"/>
       </geometry>
       <material name="pg36_shaft_material">
@@ -119,5 +119,5 @@
       <origin xyz="0 -0.007 -0.023" rpy="1.5708 -1.5708 0"/>
       <geometry>
-        <mesh filename="package://amrbot_description/meshes/pg36_shaft.stl"/>
+        <mesh filename="package://${package_name}/meshes/pg36_shaft.stl"/>
       </geometry>
     </collision>
@@ -134,5 +134,5 @@
       <origin xyz="0 0 0" rpy="1.5708 -0 0"/>
       <geometry>
-        <mesh filename="package://amrbot_description/meshes/wheel.stl"/>
+        <mesh filename="package://${package_name}/meshes/wheel.stl"/>
       </geometry>
       <material name="wheel_material">
@@ -143,5 +143,5 @@
       <origin xyz="0 0 0" rpy="1.5708 -0 0"/>
       <geometry>
-        <mesh filename="package://amrbot_description/meshes/wheel.stl"/>
+        <mesh filename="package://${package_name}/meshes/wheel.stl"/>
       </geometry>
     </collision>
@@ -150,5 +150,5 @@
       <origin xyz="0 0 0" rpy="1.5708 -0 0"/>
       <geometry>
-        <mesh filename="package://amrbot_description/meshes/tyre.stl"/>
+        <mesh filename="package://${package_name}/meshes/tyre.stl"/>
       </geometry>
       <material name="tyre_material">
@@ -159,5 +159,5 @@
       <origin xyz="0 0 0" rpy="1.5708 -0 0"/>
       <geometry>
-        <mesh filename="package://amrbot_description/meshes/tyre.stl"/>
+        <mesh filename="package://${package_name}/meshes/tyre.stl"/>
       </geometry>
     </collision>
@@ -166,5 +166,5 @@
       <origin xyz="0 0 0" rpy="1.5708 -0 0"/>
       <geometry>
-        <mesh filename="package://amrbot_description/meshes/8mm_flange_hub.stl"/>
+        <mesh filename="package://${package_name}/meshes/8mm_flange_hub.stl"/>
       </geometry>
       <material name="8mm_flange_hub_material">
@@ -175,5 +175,5 @@
       <origin xyz="0 0 0" rpy="1.5708 -0 0"/>
       <geometry>
-        <mesh filename="package://amrbot_description/meshes/8mm_flange_hub.stl"/>
+        <mesh filename="package://${package_name}/meshes/8mm_flange_hub.stl"/>
       </geometry>
     </collision>
@@ -206,5 +206,5 @@
       <origin xyz="0 -0.007 -0.023" rpy="1.5708 -1.5708 0"/>
       <geometry>
-        <mesh filename="package://amrbot_description/meshes/pg36_body.stl"/>
+        <mesh filename="package://${package_name}/meshes/pg36_body.stl"/>
       </geometry>
       <material name="pg36_body_2_material">
@@ -215,5 +215,5 @@
       <origin xyz="0 -0.007 -0.023" rpy="1.5708 -1.5708 0"/>
       <geometry>
-        <mesh filename="package://amrbot_description/meshes/pg36_body.stl"/>
+        <mesh filename="package://${package_name}/meshes/pg36_body.stl"/>
       </geometry>
     </collision>
@@ -222,5 +222,5 @@
       <origin xyz="0 -0.0072 -0.023" rpy="-1.5708 -0 0"/>
       <geometry>
-        <mesh filename="package://amrbot_description/meshes/bracket_body.stl"/>
+        <mesh filename="package://${package_name}/meshes/bracket_body.stl"/>
       </geometry>
       <material name="bracket_body_2_material">
@@ -231,5 +231,5 @@
       <origin xyz="0 -0.0072 -0.023" rpy="-1.5708 -0 0"/>
       <geometry>
-        <mesh filename="package://amrbot_description/meshes/bracket_body.stl"/>
+        <mesh filename="package://${package_name}/meshes/bracket_body.stl"/>
       </geometry>
     </collision>
@@ -238,5 +238,5 @@
       <origin xyz="0 -0.01 -0.023" rpy="-1.5708 -0 0"/>
       <geometry>
-        <mesh filename="package://amrbot_description/meshes/bracket_shaft.stl"/>
+        <mesh filename="package://${package_name}/meshes/bracket_shaft.stl"/>
       </geometry>
       <material name="bracket_shaft_2_material">
@@ -247,5 +247,5 @@
       <origin xyz="0 -0.01 -0.023" rpy="-1.5708 -0 0"/>
       <geometry>
-        <mesh filename="package://amrbot_description/meshes/bracket_shaft.stl"/>
+        <mesh filename="package://${package_name}/meshes/bracket_shaft.stl"/>
       </geometry>
     </collision>
@@ -254,5 +254,5 @@
       <origin xyz="0 -0.007 -0.023" rpy="1.5708 -1.5708 0"/>
       <geometry>
-        <mesh filename="package://amrbot_description/meshes/pg36_shaft.stl"/>
+        <mesh filename="package://${package_name}/meshes/pg36_shaft.stl"/>
       </geometry>
       <material name="pg36_shaft_2_material">
@@ -263,5 +263,5 @@
       <origin xyz="0 -0.007 -0.023" rpy="1.5708 -1.5708 0"/>
       <geometry>
-        <mesh filename="package://amrbot_description/meshes/pg36_shaft.stl"/>
+        <mesh filename="package://${package_name}/meshes/pg36_shaft.stl"/>
       </geometry>
     </collision>
@@ -278,5 +278,5 @@
       <origin xyz="0 0 0.003" rpy="1.5708 -0 0"/>
       <geometry>
-        <mesh filename="package://amrbot_description/meshes/wheel.stl"/>
+        <mesh filename="package://${package_name}/meshes/wheel.stl"/>
       </geometry>
       <material name="wheel_2_material">
@@ -287,5 +287,5 @@
       <origin xyz="0 0 0.003" rpy="1.5708 -0 0"/>
       <geometry>
-        <mesh filename="package://amrbot_description/meshes/wheel.stl"/>
+        <mesh filename="package://${package_name}/meshes/wheel.stl"/>
       </geometry>
     </collision>
@@ -294,5 +294,5 @@
       <origin xyz="0 0 0.003" rpy="1.5708 -0 0"/>
       <geometry>
-        <mesh filename="package://amrbot_description/meshes/tyre.stl"/>
+        <mesh filename="package://${package_name}/meshes/tyre.stl"/>
       </geometry>
       <material name="tyre_2_material">
@@ -303,5 +303,5 @@
       <origin xyz="0 0 0.003" rpy="1.5708 -0 0"/>
       <geometry>
-        <mesh filename="package://amrbot_description/meshes/tyre.stl"/>
+        <mesh filename="package://${package_name}/meshes/tyre.stl"/>
       </geometry>
     </collision>
@@ -310,5 +310,5 @@
       <origin xyz="0 0 0.003" rpy="1.5708 -0 0"/>
       <geometry>
-        <mesh filename="package://amrbot_description/meshes/8mm_flange_hub.stl"/>
+        <mesh filename="package://${package_name}/meshes/8mm_flange_hub.stl"/>
       </geometry>
       <material name="8mm_flange_hub_2_material">
@@ -319,5 +319,5 @@
       <origin xyz="0 0 0.003" rpy="1.5708 -0 0"/>
       <geometry>
-        <mesh filename="package://amrbot_description/meshes/8mm_flange_hub.stl"/>
+        <mesh filename="package://${package_name}/meshes/8mm_flange_hub.stl"/>
       </geometry>
     </collision>
@@ -350,5 +350,5 @@
       <origin xyz="0 0.0135 -0.04825" rpy="0 -0 0"/>
       <geometry>
-        <mesh filename="package://amrbot_description/meshes/caster_frame.stl"/>
+        <mesh filename="package://${package_name}/meshes/caster_frame.stl"/>
       </geometry>
       <material name="caster_frame_material">
@@ -359,5 +359,5 @@
       <origin xyz="0 0.0135 -0.04825" rpy="0 -0 0"/>
       <geometry>
-        <mesh filename="package://amrbot_description/meshes/caster_frame.stl"/>
+        <mesh filename="package://${package_name}/meshes/caster_frame.stl"/>
       </geometry>
     </collision>
@@ -374,5 +374,5 @@
       <origin xyz="0 0 0" rpy="1.5708 -0 0"/>
       <geometry>
-        <mesh filename="package://amrbot_description/meshes/caster_wheel.stl"/>
+        <mesh filename="package://${package_name}/meshes/caster_wheel.stl"/>
       </geometry>
       <material name="caster_wheel_material">
@@ -383,5 +383,5 @@
       <origin xyz="0 0 0" rpy="1.5708 -0 0"/>
       <geometry>
-        <mesh filename="package://amrbot_description/meshes/caster_wheel.stl"/>
+        <mesh filename="package://${package_name}/meshes/caster_wheel.stl"/>
       </geometry>
     </collision>
@@ -414,5 +414,5 @@
       <origin xyz="0 0.0135 -0.04825" rpy="0 -0 0"/>
       <geometry>
-        <mesh filename="package://amrbot_description/meshes/caster_frame.stl"/>
+        <mesh filename="package://${package_name}/meshes/caster_frame.stl"/>
       </geometry>
       <material name="caster_frame_2_material">
@@ -423,5 +423,5 @@
       <origin xyz="0 0.0135 -0.04825" rpy="0 -0 0"/>
       <geometry>
-        <mesh filename="package://amrbot_description/meshes/caster_frame.stl"/>
+        <mesh filename="package://${package_name}/meshes/caster_frame.stl"/>
       </geometry>
     </collision>
@@ -438,5 +438,5 @@
       <origin xyz="0 0 0" rpy="1.5708 -0 0"/>
       <geometry>
-        <mesh filename="package://amrbot_description/meshes/caster_wheel.stl"/>
+        <mesh filename="package://${package_name}/meshes/caster_wheel.stl"/>
       </geometry>
       <material name="caster_wheel_2_material">
@@ -447,5 +447,5 @@
       <origin xyz="0 0 0" rpy="1.5708 -0 0"/>
       <geometry>
-        <mesh filename="package://amrbot_description/meshes/caster_wheel.stl"/>
+        <mesh filename="package://${package_name}/meshes/caster_wheel.stl"/>
       </geometry>
     </collision>
@@ -478,5 +478,5 @@
       <origin xyz="0 0.0135 -0.04825" rpy="0 -0 0"/>
       <geometry>
-        <mesh filename="package://amrbot_description/meshes/caster_frame.stl"/>
+        <mesh filename="package://${package_name}/meshes/caster_frame.stl"/>
       </geometry>
       <material name="caster_frame_3_material">
@@ -487,5 +487,5 @@
       <origin xyz="0 0.0135 -0.04825" rpy="0 -0 0"/>
       <geometry>
-        <mesh filename="package://amrbot_description/meshes/caster_frame.stl"/>
+        <mesh filename="package://${package_name}/meshes/caster_frame.stl"/>
       </geometry>
     </collision>
@@ -502,5 +502,5 @@
       <origin xyz="0 0 -0.027" rpy="-1.5708 -0 0"/>
       <geometry>
-        <mesh filename="package://amrbot_description/meshes/caster_wheel.stl"/>
+        <mesh filename="package://${package_name}/meshes/caster_wheel.stl"/>
       </geometry>
       <material name="caster_wheel_3_material">
@@ -511,5 +511,5 @@
       <origin xyz="0 0 -0.027" rpy="-1.5708 -0 0"/>
       <geometry>
-        <mesh filename="package://amrbot_description/meshes/caster_wheel.stl"/>
+        <mesh filename="package://${package_name}/meshes/caster_wheel.stl"/>
       </geometry>
     </collision>
@@ -542,5 +542,5 @@
       <origin xyz="0 0.0135 -0.04825" rpy="0 -0 0"/>
       <geometry>
-        <mesh filename="package://amrbot_description/meshes/caster_frame.stl"/>
+        <mesh filename="package://${package_name}/meshes/caster_frame.stl"/>
       </geometry>
       <material name="caster_frame_4_material">
@@ -551,5 +551,5 @@
       <origin xyz="0 0.0135 -0.04825" rpy="0 -0 0"/>
       <geometry>
-        <mesh filename="package://amrbot_description/meshes/caster_frame.stl"/>
+        <mesh filename="package://${package_name}/meshes/caster_frame.stl"/>
       </geometry>
     </collision>
@@ -566,5 +566,5 @@
       <origin xyz="0 0 -0.027" rpy="-1.5708 -0 0"/>
       <geometry>
-        <mesh filename="package://amrbot_description/meshes/caster_wheel.stl"/>
+        <mesh filename="package://${package_name}/meshes/caster_wheel.stl"/>
       </geometry>
       <material name="caster_wheel_4_material">
@@ -575,5 +575,5 @@
       <origin xyz="0 0 -0.027" rpy="-1.5708 -0 0"/>
       <geometry>
-        <mesh filename="package://amrbot_description/meshes/caster_wheel.stl"/>
+        <mesh filename="package://${package_name}/meshes/caster_wheel.stl"/>
       </geometry>
     </collision>

File: src/amrbot_description/urdf/modules/imu.xacro (robot description, xacro)
@@ -12,5 +12,5 @@
       <origin xyz="-0 0 -0.01" rpy="0 -0 0"/>
       <geometry>
-        <mesh filename="package://amrbot_description/meshes/imu.stl"/>
+        <mesh filename="package://${package_name}/meshes/imu.stl"/>
       </geometry>
       <material name="imu_material">
@@ -21,5 +21,5 @@
       <origin xyz="-0 0 -0.01" rpy="0 -0 0"/>
       <geometry>
-        <mesh filename="package://amrbot_description/meshes/imu.stl"/>
+        <mesh filename="package://${package_name}/meshes/imu.stl"/>
       </geometry>
     </collision>

File: src/amrbot_description/urdf/modules/lidar.xacro (robot description, xacro)
@@ -12,5 +12,5 @@
       <origin xyz="0 -0 0.069" rpy="3.14159 -0 0"/>
       <geometry>
-        <mesh filename="package://amrbot_description/meshes/electrical_box.stl"/>
+        <mesh filename="package://${package_name}/meshes/electrical_box.stl"/>
       </geometry>
       <material name="electrical_box_material">
@@ -21,5 +21,5 @@
       <origin xyz="0 -0 0.069" rpy="3.14159 -0 0"/>
       <geometry>
-        <mesh filename="package://amrbot_description/meshes/electrical_box.stl"/>
+        <mesh filename="package://${package_name}/meshes/electrical_box.stl"/>
       </geometry>
     </collision>
@@ -36,5 +36,5 @@
       <origin xyz="0.000613921 -0.000614591 0" rpy="3.14159 -0 0"/>
       <geometry>
-        <mesh filename="package://amrbot_description/meshes/lidar.stl"/>
+        <mesh filename="package://${package_name}/meshes/lidar.stl"/>
       </geometry>
       <material name="lidar_material">
@@ -45,5 +45,5 @@
       <origin xyz="0.000613921 -0.000614591 0" rpy="3.14159 -0 0"/>
       <geometry>
-        <mesh filename="package://amrbot_description/meshes/lidar.stl"/>
+        <mesh filename="package://${package_name}/meshes/lidar.stl"/>
       </geometry>
     </collision>
