Commit message: Modify files

File: src/amrbot_description/urdf/ros2_control/amrbot.ros2_control.xacro (robot description, xacro)
@@ -5,10 +5,10 @@
       <plugin>amrbot_hardware/AmrbotHardwareInterface</plugin>
     </hardware>
-    <joint name="wheel_left_joint">
+    <joint name="left_wheel_joint">
       <command_interface name="velocity"/>
       <state_interface name="position"/>
       <state_interface name="velocity"/>
     </joint>
-    <joint name="wheel_right_joint">
+    <joint name="right_wheel_joint">
       <command_interface name="velocity"/>
       <state_interface name="position"/>
